Commit message: Remove igni diff drive

File: src/diffdrive_description/urdf/robot.urdf.xacro (robot description, xacro)
@@ -31,5 +31,5 @@
         <parent link="base_footprint" />
         <child link="base_link" />
-        <origin xyz="0.0 0.0  ${wheel_radius + base_height/2}" rpy="0 0 0" />
+        <origin xyz="0.0 0.0  ${wheel_radius + base_height/2 - wheel_zoff}" rpy="0 0 0" />
     </joint>
     <xacro:macro name="wheel" params="prefix x_reflect y_reflect">
@@ -88,23 +88,4 @@
         <mu2>0.001</mu2>
     </gazebo>
-    <gazebo>
-        <plugin filename="libignition-gazebo-diff-drive-system.so" name="ignition::gazebo::systems::DiffDrive">
-            <left_joint>drivewhl_l_joint</left_joint>
-            <right_joint>drivewhl_r_joint</right_joint>
-            <wheel_separation>1.2</wheel_separation>
-            <wheel_radius>0.1</wheel_radius>
-            <odom_publish_frequency>30</odom_publish_frequency>
-            <frame_id>odom</frame_id>
-            <child_frame_id>base_footprint</child_frame_id>
-            <odom_topic>odom</odom_topic>
-            <topic>cmd_vel</topic>
-            <tf_topic>tf</tf_topic>
-        </plugin>
-        <plugin filename="gz-sim-joint-state-publisher-system" name="gz::sim::systems::JointStatePublisher">
-            <topic>joint_states</topic>
-            <joint_name>drivewhl_l_joint</joint_name>
-            <joint_name>drivewhl_r_joint</joint_name>
-        </plugin>
-    </gazebo>
     <link name="imu_link">
         <visual>

Commit message: Add ros2 conntrol to urdf

File: src/diffdrive_description/urdf/robot.urdf.xacro (robot description, xacro)
@@ -63,4 +63,34 @@
     <xacro:wheel prefix="drivewhl_l" x_reflect="-1" y_reflect="1" />
     <xacro:wheel prefix="drivewhl_r" x_reflect="-1" y_reflect="-1" />
+    <ros2_control name="IgnitionSystem" type="system">
+        <hardware>
+        <plugin>ign_ros2_control/IgnitionSystem</plugin>
+        </hardware>
+        <joint name="drivewhl_l_joint">
+        <command_interface name="velocity">
+            <param name="min">-1</param>
+            <param name="max">1</param>
+        </command_interface>
+        <state_interface name="position"/>
+        <state_interface name="velocity"/>
+        </joint>
+        <joint name="drivewhl_r_joint">
+        <command_interface name="velocity">
+            <param name="min">-1</param>
+            <param name="max">1</param>
+        </command_interface>
+        <state_interface name="position"/>
+        <state_interface name="velocity"/>
+        </joint>
+    </ros2_control>
+    <gazebo>
+        <plugin filename="ign_ros2_control-system" name="ign_ros2_control::IgnitionROS2ControlPlugin">
+            <parameters>$(find diffdrive_bringup)/config/controllers.yaml</parameters>
+            <ros>
+                <remapping>/diff_drive_controller/cmd_vel_unstamped:=/cmd_vel</remapping>
+                <remapping>/diff_drive_controller/odom:=/odom</remapping>
+            </ros>
+        </plugin>
+    </gazebo>
     <link name="front_caster">
         <visual>
@@ -108,9 +138,10 @@
     <gazebo reference="imu_link">
         <sensor name="imu_sensor" type="imu">
-            <plugin filename="libignition-gazebo-imu-system.so" name="ignition::gazebo::systems::Imu" />
+            <plugin filename="libignition-gazebo-imu-system.so" name="ignition::gazebo::systems::Imu"/>
             <always_on>1</always_on>
             <update_rate>10</update_rate>
             <visualize>true</visualize>
             <topic>imu</topic>
+            <gz_frame_id>imu_link</gz_frame_id>
         </sensor>
     </gazebo>

Commit message: Add change to diffdrive gazebo plugin

File: src/diffdrive_description/urdf/robot.urdf.xacro (robot description, xacro)
@@ -63,32 +63,22 @@
     <xacro:wheel prefix="drivewhl_l" x_reflect="-1" y_reflect="1" />
     <xacro:wheel prefix="drivewhl_r" x_reflect="-1" y_reflect="-1" />
-    <ros2_control name="IgnitionSystem" type="system">
-        <hardware>
-        <plugin>ign_ros2_control/IgnitionSystem</plugin>
-        </hardware>
-        <joint name="drivewhl_l_joint">
-        <command_interface name="velocity">
-            <param name="min">-1</param>
-            <param name="max">1</param>
-        </command_interface>
-        <state_interface name="position"/>
-        <state_interface name="velocity"/>
-        </joint>
-        <joint name="drivewhl_r_joint">
-        <command_interface name="velocity">
-            <param name="min">-1</param>
-            <param name="max">1</param>
-        </command_interface>
-        <state_interface name="position"/>
-        <state_interface name="velocity"/>
-        </joint>
-    </ros2_control>
     <gazebo>
-        <plugin filename="ign_ros2_control-system" name="ign_ros2_control::IgnitionROS2ControlPlugin">
-            <parameters>$(find diffdrive_bringup)/config/controllers.yaml</parameters>
-            <ros>
-                <remapping>/diff_drive_controller/cmd_vel_unstamped:=/cmd_vel</remapping>
-                <remapping>/diff_drive_controller/odom:=/odom</remapping>
-            </ros>
+        <plugin filename="gz-sim-diff-drive-system" name="gz::sim::systems::DiffDrive">
+            <left_joint>drivewhl_l_joint</left_joint>
+            <right_joint>drivewhl_r_joint</right_joint>
+            <wheel_separation>0.4</wheel_separation>
+            <wheel_radius>0.1</wheel_radius>
+            <max_linear_acceleration>0.2</max_linear_acceleration>
+            <topic>cmd_vel</topic>
+            <odom_topic>odom</odom_topic>
+            <frame_id>odom</frame_id>
+            <child_frame_id>base_footprint</child_frame_id>
+            <odom_publisher_frequency>30</odom_publisher_frequency>
+            <tf_topic>/tf</tf_topic>
+        </plugin>
+        <plugin filename="gz-sim-joint-state-publisher-system" name="gz::sim::systems::JointStatePublisher">
+            <topic>joint_states</topic>
+            <joint_name>drivewhl_l_joint</joint_name>
+            <joint_name>drivewhl_r_joint</joint_name>
         </plugin>
     </gazebo>
